File: bmp clone.kicad_sch (KiCad schematic)
At the start: 46 parts, among them J1 Conn_02x10_Odd_Even, J3 Jumper_2_Open, P1 USB_C_Plug_USB2.0, Q1 BC846, U1 STM32F103RBTx, U2 USBLC6-2P6, U3 TXS0108EPW, U4 AMS1117-3.3, X1 8MHz

Commit message: pcb
Parts:
- removed C11, C12, C13: 100n, Capacitor_SMD:C_0805_2012Metric, symbol Device:C
- removed P1: USB_C_Plug_USB2.0, Connector_USB:USB_C_Plug_JAE_DX07P024AJ1, symbol Connector:USB_C_Plug_USB2.0
- removed R14: 1k, Resistor_SMD:R_0805_2012Metric, symbol Device:R
- removed S1: SW_MEC_5G, Button_Switch_SMD:SW_DIP_SPSTx01_Slide_Copal_CHS-01A_W5.08mm_P1.27mm_JPin, symbol Switch:SW_MEC_5G
- added J2: USB_B_Mini, Connector_USB:USB_Mini-B_Lumberg_2486_01_Horizontal, symbol Connector:USB_B_Mini
- J1: footprint Connector_IDC:IDC-Header_2x08_P2.54mm_Horizontal -> Connector_IDC:IDC-Header_2x08_P2.54mm_Vertical
- X1: footprint Crystal:Crystal_HC49-4H_Vertical -> Crystal:Crystal_SMD_3225-4Pin_3.2x2.5mm
Connections:
- net +5V: now also J2.1 (VBUS)
- net GND: now also J2.5 (GND), J2.6 (Shield)
- net at U2.1 (I/O1): now also J2.2 (D-)
- net at U2.3 (I/O2): now also J2.3 (D+)
- no-connect marks 34 -> 33

Commit message: dodani su gerberi i preza
Other:
- note added: "LED diode za dijagnostiku"
- note added: "Linearni regulator (3,3 V)"
- note added: "Mikrokontroler"
- note added: "Pretvarač napona"
- note added: "USB micro B i ESD zaštita"
- moved on the sheet: C3, C4, D1, D2, D3, D4, R10, R11, R12, R13, R5, R6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
