File: bmp clone.kicad_pcb (KiCad board)
At the start: 2 copper layers, 56.5 x 29.8 mm, 46 parts, among them J1 Conn_02x10_Odd_Even, J3 Jumper_2_Open, P1 USB_C_Plug_USB2.0, Q1 BC846, U1 STM32F103RBTx, U2 USBLC6-2P6, U3 TXS0108EPW, U4 AMS1117-3.3, X1 8MHz

Commit message: pcb
Parts:
- removed C11, C12, C13: 100n, Capacitor_SMD:C_0805_2012Metric
- removed P1: USB_C_Plug_USB2.0, Connector_USB:USB_C_Plug_JAE_DX07P024AJ1
- removed R14: 1k, Resistor_SMD:R_0805_2012Metric
- removed S1: SW_MEC_5G, Button_Switch_SMD:SW_DIP_SPSTx01_Slide_Copal_CHS-01A_W5.08mm_P1.27mm_JPin
- added J2: USB_B_Mini, Connector_USB:USB_Mini-B_Lumberg_2486_01_Horizontal, F.Cu at (117.5, 90.9)
- J1: footprint Connector_IDC:IDC-Header_2x08_P2.54mm_Horizontal -> Connector_IDC:IDC-Header_2x08_P2.54mm_Vertical
- X1: footprint Crystal:Crystal_HC49-4H_Vertical -> Crystal:Crystal_SMD_3225-4Pin_3.2x2.5mm
- moved U3 48.5 mm to (151.9, 93.2)
- moved R5 44.1 mm to (143.7, 101.6), turned to 0 degrees
- moved R15 42.9 mm to (147.6, 88.7)
- moved D2 41.1 mm to (137.3, 78.3)
- moved D3 41.1 mm to (139.6, 78.3)
- moved R10 41.1 mm to (139.6, 82.3)
- moved R9 41.1 mm to (137.3, 82.3)
- moved D4 41.1 mm to (141.9, 78.3)
- moved LED 41.1 mm to (135.0, 78.3)
- moved R8 41.1 mm to (135.0, 82.3)
- moved R11 41.1 mm to (141.9, 82.3)
- moved TP1 40.2 mm to (137.5, 88.5)
- moved TP2 39.8 mm to (134.1, 88.5)
- moved J1 39.3 mm to (160.1, 82.3)
- moved U1 38.8 mm to (137.4, 91.8), turned to 90 degrees
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- renumbered D1 to LED
Connections:
- U1 pad 33: Net-(U1-PB12) -> unconnected-(U1-PB12-Pad33)
Routing:
- net /BOOT_0: track 26.7 -> 61.7 mm
- net /U1RX: track 0.00 -> 32.1 mm, vias 0 -> 1
- net /U1TX: track 0.00 -> 31.4 mm, vias 0 -> 1
- net GND: track 60.6 -> 32.9 mm, vias 18 -> 37
- net +3.3V: track 89.9 -> 110.3 mm, vias 2 -> 0
- net Net-(J1-Pin_1): track 17.8 -> 36.9 mm
- net /xTDI: track 0.00 -> 15.4 mm
- net /xnSRST_OUT: track 4.50 -> 18.5 mm, vias 0 -> 2
- net /xnTRST: track 19.8 -> 6.10 mm, vias 2 -> 0
- net /USB_DP: track 14.3 -> 26.5 mm
- net /USB_PU: track 7.95 -> 18.9 mm
- net /USB_DM: track 7.90 -> 17.0 mm, vias 0 -> 2
- net Net-(U1-PB12): track 8.71 -> 0.00 mm
- net Net-(J1-Pin_3): track 0.00 -> 8.71 mm
- net /LED_0: track 6.39 -> 14.4 mm, vias 0 -> 2
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- added copper zone on F.Cu, net +3.3V
- added copper zone on F.Cu, net GND
Other:
- board size 56.5 x 29.8 mm -> 55 x 31 mm
- board text added: "Black Magic probe clone"
- board text added: "Jadran Marinović TVZ - 2024"

Commit message: dodani su gerberi i preza
Changed lines of the file:
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@@
 			(psnegative no)
 			(psa4output no)
-			(plotreference yes)
-			(plotvalue yes)
-			(plotfptext yes)
+			(plotreference no)
+			(plotvalue no)
+			(plotfptext no)
 			(plotinvisibletext no)
 			(sketchpadsonfab no)
@@
 			(drillshape 0)
 			(scaleselection 1)
-			(outputdirectory "../../pcb git/")
+			(outputdirectory "gerberi/")
 		)
 	)
@@
 	)
 	(gr_text "Black Magic \nprobe clone\n"
-		(at 145.4 105.3 0)
+		(at 146.4 103.475 0)
 		(layer "F.SilkS")
 		(effects
@@
 		(polygon
 			(pts
-				(xy 116.2 88.15) (xy 121.55 88.15) (xy 121.55 94.525) (xy 123.35 94.525) (xy 123.4 99.825) (xy 116.15 99.825)
+				(xy 116.2 88.15) (xy 121.55 88.15) (xy 121.55 95.025) (xy 124.4 95.025) (xy 124.4 99.825) (xy 116.15 99.825)
 			)
 		)
@@
 			)
 		)
-	)
-	(zone
-		(net 5)
-		(net_name "+5V")
-		(layer "F.Cu")
-		(hatch edge 0.5)
-		(priority 5)
-		(connect_pads yes
-			(clearance 0.5)
-		)
-		(min_thickness 0.25)
-		(filled_areas_thickness no)
-		(fill yes
-			(thermal_gap 0.5)
-			(thermal_bridge_width 0.5)
-		)
-		(polygon
-			(pts
-				(xy 124.5 99.8) (xy 124.5 95.4) (xy 122.9 95.4) (xy 122.9 97.9) (xy 119.8 97.9) (xy 119.8 99.8)
-			)
-		)

Commit message: manje dorade
Routing:
- net +3.3V: track 110.3 -> 110.9 mm
Changed lines of the file:
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@@
-	)
-	(segment
-		(start 134.2 92.8)
-		(end 132.9 91.5)
-		(width 0.3)
-		(layer "F.Cu")
-		(net 6)
 	)
 	(segment
@@
 	)
 	(segment
+		(start 134.2 92.175)
+		(end 134.2 91.975)
+		(width 0.3)
+		(layer "F.Cu")
+		(net 6)
+	)
+	(segment
 		(start 140.339852 94.2)
 		(end 141.9 95.760148)
@@
 		(start 143.125 94.5)
 		(end 145.25 94.5)
+		(width 0.3)
+		(layer "F.Cu")
+		(net 6)
+	)
+	(segment
+		(start 134.2 92.8)
+		(end 133.8875 92.4875)
 		(width 0.3)
 		(layer "F.Cu")
@@
 	)
 	(segment
+		(start 133.8875 92.4875)
+		(end 134.2 92.175)
+		(width 0.3)
+		(layer "F.Cu")
+		(net 6)
+	)
+	(segment
 		(start 134.2 90.1)
 		(end 133.7 89.6)
@@
 	)
 	(segment
+		(start 134.2 92.8)
+		(end 134.2 91.975)
+		(width 0.3)
+		(layer "F.Cu")
+		(net 6)
+	)
+	(segment
 		(start 123.7 104.2)
 		(end 123.7 101.6)
@@
 	)
 	(segment
+		(start 133.8875 92.4875)
+		(end 132.9 91.5)
+		(width 0.3)
+		(layer "F.Cu")
+		(net 6)
+	)
+	(segment
 		(start 128.2 98)
 		(end 128.2 97.975)
@@
 	)
 	(segment
-		(start 134.2 92.8)
-		(end 134.2 90.1)
-		(width 0.3)
-		(layer "F.Cu")
-		(net 6)
-	)
-	(segment
 		(start 128.344544 94.5375)
 		(end 129.93438 94.5375)
@@
 		(start 133.7 95.5)
 		(end 134.2 95)
+		(width 0.3)
+		(layer "F.Cu")
+		(net 6)
+	)
+	(segment
+		(start 134.2 91.975)
+		(end 134.2 90.1)
 		(width 0.3)
 		(layer "F.Cu")
@@
 	)
 	(segment
-		(start 144.42 82.28)
-		(end 149.55 77.15)
+		(start 130.4375 96.1)
+		(end 134.1 96.1)
+		(width 0.3)
+		(layer "F.Cu")
+		(net 14)
+	)
+	(segment
+		(start 142.2 86.45312)
+		(end 142.2 85.55)
+		(width 0.3)
+		(layer "F.Cu")
+		(net 14)
+	)
+	(segment
+		(start 134.9 95.3)
+		(end 138.6 95.3)
+		(width 0.3)
+		(layer "F.Cu")
+		(net 14)
+	)
+	(segment
+		(start 139 88.8)
+		(end 140.6 87.2)
+		(width 0.3)
+		(layer "F.Cu")
+		(net 14)
+	)
+	(segment
+		(start 140.75 84.1)
+		(end 140.75 82.65)
 		(width 0.3)
 		(layer "F.Cu")
@@
 	)
 	(segment
+		(start 160.15 77.15)
+		(end 164.4 81.4)
+		(width 0.3)
+		(layer "F.Cu")
+		(net 14)
+	)
+	(segment
+		(start 141.45312 87.2)
+		(end 142.2 86.45312)
+		(width 0.3)
+		(layer "F.Cu")
+		(net 14)
+	)
+	(segment
+		(start 143.845 82.28)
+		(end 148.975 77.15)
+		(width 0.3)
+		(layer "F.Cu")
+		(net 14)
+	)
+	(segment
+		(start 129.75 95.4125)
+		(end 130.4375 96.1)
+		(width 0.3)
+		(layer "F.Cu")
+		(net 14)
+	)
+	(segment
+		(start 134.1 96.1)
+		(end 134.9 95.3)
+		(width 0.3)
+		(layer "F.Cu")
+		(net 14)
+	)
+	(segment
+		(start 142.2 85.55)
+		(end 140.75 84.1)
+		(width 0.3)
+		(layer "F.Cu")
+		(net 14)
+	)
+	(segment
+		(start 148.975 77.15)
+		(end 160.15 77.15)
+		(width 0.3)
+		(layer "F.Cu")
+		(net 14)
+	)
+	(segment
+		(start 164.4 81.4)
+		(end 164.4 88.1725)
+		(width 0.3)
+		(layer "F.Cu")
+		(net 14)
+	)
+	(segment
+		(start 140.6 87.2)
+		(end 141.45312 87.2)
+		(width 0.3)
+		(layer "F.Cu")
+		(net 14)
+	)
+	(segment
+		(start 140.75 82.65)
+		(end 141.12 82.28)
+		(width 0.3)
+		(layer "F.Cu")
+		(net 14)
+	)
+	(segment
 		(start 138.6 95.3)
 		(end 139 94.9)
@@
 	)
 	(segment
-		(start 129.75 95.4125)
-		(end 130.4375 96.1)
-		(width 0.3)
-		(layer "F.Cu")
-		(net 14)
-	)
-	(segment
-		(start 140.75 84.1)
-		(end 140.75 82.65)
-		(width 0.3)
-		(layer "F.Cu")
-		(net 14)
-	)
-	(segment
-		(start 134.9 95.3)
-		(end 138.6 95.3)
-		(width 0.3)
-		(layer "F.Cu")
-		(net 14)
-	)
-	(segment
-		(start 164.4 81.4)
-		(end 164.4 88.1725)
-		(width 0.3)
-		(layer "F.Cu")
-		(net 14)
-	)
-	(segment
-		(start 134.1 96.1)
-		(end 134.9 95.3)
-		(width 0.3)
-		(layer "F.Cu")
-		(net 14)
-	)
-	(segment
-		(start 141.45312 87.2)
-		(end 142.2 86.45312)
-		(width 0.3)
-		(layer "F.Cu")
-		(net 14)
-	)
-	(segment
-		(start 140.6 87.2)
-		(end 141.45312 87.2)
-		(width 0.3)
-		(layer "F.Cu")
-		(net 14)
-	)
-	(segment
-		(start 130.4375 96.1)
-		(end 134.1 96.1)
-		(width 0.3)
-		(layer "F.Cu")
-		(net 14)
-	)
-	(segment
-		(start 142.2 85.55)
-		(end 140.75 84.1)
-		(width 0.3)
-		(layer "F.Cu")
-		(net 14)
-	)
-	(segment
-		(start 160.15 77.15)
-		(end 164.4 81.4)
-		(width 0.3)
-		(layer "F.Cu")
-		(net 14)
-	)
-	(segment
-		(start 141.12 82.28)
-		(end 144.42 82.28)
-		(width 0.3)
-		(layer "F.Cu")
-		(net 14)
-	)
-	(segment
 		(start 164.4 88.1725)
 		(end 162.6425 89.93)
@@
 	)
 	(segment
-		(start 140.75 82.65)
-		(end 141.12 82.28)
-		(width 0.3)
-		(layer "F.Cu")
-		(net 14)
-	)
-	(segment
-		(start 142.2 86.45312)
-		(end 142.2 85.55)
-		(width 0.3)
-		(layer "F.Cu")
-		(net 14)
-	)
-	(segment
-		(start 149.55 77.15)
-		(end 160.15 77.15)
-		(width 0.3)
-		(layer "F.Cu")
-		(net 14)
-	)
-	(segment
-		(start 139 88.8)
-		(end 140.6 87.2)
-		(width 0.3)
-		(layer "F.Cu")
+		(start 141.12 82.28)
+		(end 143.845 82.28)
+		(width 0.3)
+		(layer "F.Cu")
